File: pcb/kicad rev7/rev7/rev7.sch (KiCad schematic (older format))
At the start: 1 part

Commit message: kicad
Parts:
- added J? (x4): 1053131103, CON_1053131103, symbol 2022-08-08_02-28-42:1053131103
- added J?: 1053131102, CON_1053131102, symbol 2022-08-08_02-26-27:1053131102
Changed lines of the file:
@@
 Wire Wire Line
 	7500 1500 7500 1900
+$Comp
+L 2022-08-08_02-28-42:1053131103 J?
+U 1 1 62F07D9F
+P 1050 1150
+F 0 "J?" H 1578 1103 60  0000 L CNN
+F 1 "1053131103" H 1578 997 60  0000 L CNN
+F 2 "CON_1053131103" H 1450 990 60  0001 C CNN
+F 3 "" H 1050 1150 60  0000 C CNN
+	1    1050 1150
+	1    0    0    -1
+$EndComp
+$Comp
+L 2022-08-08_02-26-27:1053131102 J?
+U 1 1 62F0F536
+P 1050 2150
+F 0 "J?" H 1578 2153 60  0000 L CNN
+F 1 "1053131102" H 1578 2047 60  0000 L CNN
+F 2 "CON_1053131102" H 1450 2090 60  0001 C CNN
+F 3 "" H 1050 2150 60  0000 C CNN
+	1    1050 2150
+	1    0    0    -1
+$EndComp
+$Comp
+L 2022-08-08_02-28-42:1053131103 J?
+U 1 1 62F1257D
+P 1050 1650
+F 0 "J?" H 1578 1603 60  0000 L CNN
+F 1 "1053131103" H 1578 1497 60  0000 L CNN
+F 2 "CON_1053131103" H 1450 1490 60  0001 C CNN
+F 3 "" H 1050 1650 60  0000 C CNN
+	1    1050 1650
+	1    0    0    -1
+$EndComp
+$Comp
+L 2022-08-08_02-28-42:1053131103 J?
+U 1 1 62F13085
+P 1050 2550
+F 0 "J?" H 1578 2503 60  0000 L CNN
+F 1 "1053131103" H 1578 2397 60  0000 L CNN
+F 2 "CON_1053131103" H 1450 2390 60  0001 C CNN
+F 3 "" H 1050 2550 60  0000 C CNN
+	1    1050 2550
+	1    0    0    -1
+$EndComp
+$Comp
+L 2022-08-08_02-28-42:1053131103 J?
+U 1 1 62F13A55
+P 1050 3050
+F 0 "J?" H 1578 3003 60  0000 L CNN
+F 1 "1053131103" H 1578 2897 60  0000 L CNN
+F 2 "CON_1053131103" H 1450 2890 60  0001 C CNN
+F 3 "" H 1050 3050 60  0000 C CNN
+	1    1050 3050
+	1    0    0    -1
+$EndComp
 $EndSCHEMATC
